File: amplificador_200w_estereo.kicad_sch (KiCad schematic)
At the start: 11 parts, among them J1 Conn_01x03, J2 input, J3 out, J4 out, J6 out, U3 L7805

Commit message: Separando las altas con resistencias de 22K
Changed lines of the file:
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@@
 (kicad_sch (version 20211123) (generator eeschema)
   (paper "A4")
+  (title_block
+    (comment 1 "${NAME}")
+  )
   (junction (at 31.75 59.69) (diameter 0) (color 0 0 0 0)
   )
@@
     )
     (path "/91c9976e-33f3-4776-850e-36ee5d251977/00000000-0000-0000-0000-000060a4ca18"
-      (reference "Q5") (unit 1) (value "BD139") (footprint "Package_TO_SOT_THT:TO-126-3_Vertical")
+      (reference "Q5") (unit 1) (value "TIP42C") (footprint "Package_TO_SOT_THT:TO-220-3_Vertical")
     )
     (path "/91c9976e-33f3-4776-850e-36ee5d251977/00000000-0000-0000-0000-000060a4ca32"
-      (reference "Q6") (unit 1) (value "BD136") (footprint "Package_TO_SOT_THT:TO-126-3_Vertical")
+      (reference "Q6") (unit 1) (value "TIP41C") (footprint "Package_TO_SOT_THT:TO-220-3_Vertical")
     )
     (path "/91c9976e-33f3-4776-850e-36ee5d251977/00000000-0000-0000-0000-000060a4ca2c"
-      (reference "Q7") (unit 1) (value "BD139") (footprint "Package_TO_SOT_THT:TO-126-3_Vertical")
+      (reference "Q7") (unit 1) (value "TIP42C") (footprint "Package_TO_SOT_THT:TO-220-3_Vertical")
     )
     (path "/91c9976e-33f3-4776-850e-36ee5d251977/00000000-0000-0000-0000-000060a4ca6f"
@@
     )
     (path "/b4ac9ced-c2e0-4836-a46e-6affbff21678/00000000-0000-0000-0000-000060a4ca18"
-      (reference "Q14") (unit 1) (value "BD139") (footprint "Package_TO_SOT_THT:TO-126-3_Vertical")
+      (reference "Q14") (unit 1) (value "TIP42C") (footprint "Package_TO_SOT_THT:TO-220-3_Vertical")
     )
     (path "/b4ac9ced-c2e0-4836-a46e-6affbff21678/00000000-0000-0000-0000-000060a4ca32"
-      (reference "Q15") (unit 1) (value "BD136") (footprint "Package_TO_SOT_THT:TO-126-3_Vertical")
+      (reference "Q15") (unit 1) (value "TIP41C") (footprint "Package_TO_SOT_THT:TO-220-3_Vertical")
     )
     (path "/b4ac9ced-c2e0-4836-a46e-6affbff21678/00000000-0000-0000-0000-000060a4ca2c"
-      (reference "Q16") (unit 1) (value "BD139") (footprint "Package_TO_SOT_THT:TO-126-3_Vertical")
+      (reference "Q16") (unit 1) (value "TIP42C") (footprint "Package_TO_SOT_THT:TO-220-3_Vertical")
     )
     (path "/b4ac9ced-c2e0-4836-a46e-6affbff21678/00000000-0000-0000-0000-000060a4ca6f"
@@
       (reference "R40") (unit 1) (value "2.7K") (footprint "Resistor_THT:R_Axial_DIN0207_L6.3mm_D2.5mm_P10.16mm_Horizontal")
     )
+    (path "/f8f15f9d-cff7-4705-91bd-f68f82997cad/0da739dc-1106-4c98-8f83-af353c76238b"
+      (reference "R41") (unit 1) (value "22K") (footprint "Resistor_THT:R_Axial_DIN0207_L6.3mm_D2.5mm_P10.16mm_Horizontal")
+    )
+    (path "/f8f15f9d-cff7-4705-91bd-f68f82997cad/99c72668-fb22-49c4-85a8-f7ffd85937ee"
+      (reference "R42") (unit 1) (value "22K") (footprint "Resistor_THT:R_Axial_DIN0207_L6.3mm_D2.5mm_P10.16mm_Horizontal")
+    )
     (path "/91c9976e-33f3-4776-850e-36ee5d251977/00000000-0000-0000-0000-000060adc9e3"

Commit message: actualizando a kicad 7
Other:
- title: (none) -> AMPLIFICADOR ESTEREO 200, CONTROL DE TONOS
