File: filtroPasaAltas.kicad_sch (KiCad schematic)
At the start: 9 parts, among them U2 TL082

Commit message: actualizando a kicad 7
Other:
- title: (none) -> AMPLIFICADOR ESTEREO 200, CONTROL DE TONOS
