File: pasa-bajo-ajust.kicad_sch (KiCad schematic)
At the start: 10 parts, among them U1 TL082

Commit message: actualizando a kicad 7
Other:
- title: Filtro pasa bajos Ajustable 30Hz a 338Hz -> AMPLIFICADOR ESTEREO 200, CONTROL DE TONOS
